Commit message: atleast motor driver working

File: blvr_diffbot_description/robots/blvr_diffbot_description.urdf.xacro (robot description, xacro)
@@ -15,5 +15,5 @@
       <type>transmission_interface/SimpleTransmission</type>
         <actuator name="${prefix}_motor">
-          <mechanicalReduction>50</mechanicalReduction>
+          <mechanicalReduction>30</mechanicalReduction>
         </actuator>
       <joint name="${prefix}_joint">
@@ -48,4 +48,11 @@
   </xacro:macro>
   <link name="base_link"/>
+<link name="laser"/>
+<joint name="laser_joint" type="fixed">
+  <parent link="body_link"/>
+  <child  link="laser"/>
+  <!-- use your real mount pose -->
+  <origin xyz="-0.14 0 0.04" rpy="0 0 0"/>
+</joint>
   <joint name="body_joint" type="fixed">
     <parent link="base_link"/>

File: blvr_diffbot_description/ros2_control/blvr_diffbot.ros2_control.xacro (robot description, xacro)
@@ -14,6 +14,6 @@
         <xacro:unless value="${use_fake_hardware or use_sim}">
           <plugin>blvr_diffbot_hardware/BlvrDiffbotSystemHardware</plugin>
-          <param name="example_param_hw_start_duration_sec">2.0</param>
-          <param name="example_param_hw_stop_duration_sec">3.0</param>
+          <param name="example_param_hw_start_duration_sec">0.0</param>
+          <param name="example_param_hw_stop_duration_sec">0.0</param>
           <param name="device_name">/dev/ttyUSB1</param>
           <param name="gear_ratio">30.0</param>

Commit message: Diff driver working

File: blvr_diffbot_description/robots/blvr_diffbot_description.urdf.xacro (robot description, xacro)
@@ -50,8 +50,8 @@
 <link name="laser"/>
 <joint name="laser_joint" type="fixed">
-  <parent link="body_link"/>
+  <parent link="base_link"/>
   <child  link="laser"/>
   <!-- use your real mount pose -->
-  <origin xyz="-0.14 0 0.04" rpy="0 0 0"/>
+  <origin xyz="0.2 0 0.04" rpy="0 0 0"/>
 </joint>
   <joint name="body_joint" type="fixed">
@@ -83,6 +83,18 @@
     <material>Gazebo/Gray</material>
   </gazebo>
-  <xacro:wheel_macro prefix="left_wheel"  parent="base_link" xyz="0 0.1 0.05"/>
-  <xacro:wheel_macro prefix="right_wheel" parent="base_link" xyz="0 -0.1 0.05"/>
+  <link name="camera_base_link"></link>
+  <link name="imu_link"></link>
+  <joint name="camera_joint" type="fixed">
+    <parent link="base_link"/>
+    <child  link="camera_base_link"/>
+    <origin xyz="0.28  0.08 0.0" rpy="0 0 0"/>
+  </joint>
+  <joint name="imu_joint" type="fixed">
+    <parent link="base_link"/>
+    <child  link="imu_link"/>
+    <origin xyz="0.0  0.0 0.0" rpy="0 0 0"/>
+  </joint>
+  <xacro:wheel_macro prefix="left_wheel"  parent="base_link" xyz="0 0.25 0.05"/>
+  <xacro:wheel_macro prefix="right_wheel" parent="base_link" xyz="0 -0.25 0.05"/>
   <joint name="ball_joint" type="fixed">
     <parent link="base_link"/>

File: blvr_diffbot_description/ros2_control/blvr_diffbot.ros2_control.xacro (robot description, xacro)
@@ -16,5 +16,5 @@
           <param name="example_param_hw_start_duration_sec">0.0</param>
           <param name="example_param_hw_stop_duration_sec">0.0</param>
-          <param name="device_name">/dev/ttyUSB1</param>
+          <param name="device_name">/dev/motor</param>
           <param name="gear_ratio">30.0</param>
           <param name="encoder_resolution">36000</param>
